Commit message: custom urdf

File: pybullet-test/torus/torus.urdf (robot description, URDF)
Before this commit: robot long_edge.urdf, 1 links, 0 joints
Links:
- removed link long_edge
- added link baseLink, mass .1; collision mesh filename=torus.obj scale=.3 .3 .3; visual mesh filename=torus.obj scale=.3 .3 .3

File: pybullet-test/torus/torus_with_plane.urdf (robot description, URDF)
Before this commit: robot long_edge.urdf, 1 links, 0 joints
Links:
- removed link long_edge
- added link baseLink, mass .1; collision mesh filename=torus_with_plane.obj scale=.3 .3 .3; visual mesh filename=torus_with_plane.obj scale=.3 .3 .3
