Commit message: follow edge test

File: pybullet-test/test.urdf (robot description, URDF)
Before this commit: robot myfirst, 1 links, 0 joints
Links:
- added link head; visual sphere radius=0.2
- added link left_leg; visual box size=0.6 0.1 0.2
- added link right_leg; visual box size=0.6 0.1 0.2
Joints:
- added joint base_to_left_leg: type fixed, parent base_link, child left_leg, origin xyz=0 0.22 0.25
- added joint base_to_right_leg: type fixed, parent base_link, child right_leg, origin xyz=0 -0.22 0.25
- added joint head_swivel: type continuous, parent base_link, child head, origin xyz=0 0 0.3, axis 0 0 1

File: tactile_gym/assets/rl_env_assets/exploration/edge_follow/edge_stimuli/long_edge_flat/cylinder_edge.urdf (robot description, URDF)
Before this commit: robot cylinder.urdf, 1 links, 0 joints
Links:
- link cylinder: geometry collision cylinder length=0.03 radius=0.15; visual cylinder length=0.03 radius=0.15
