Commit message: Added Digitac, and trained it with UR5 and MG400 in the edge task.

File: tactile_gym/assets/robot_assets/mg400/mg400_with_standard_digitac.urdf (robot description, URDF)
Before this commit: robot mg400, 13 links, 12 joints
Links:
- removed link digit_body_link
- removed link digit_tip_link
- added link digitac_body_link, mass 0.00791827593084163; collision mesh filename=../digitac/standard_digitac/digitac_asmb/meshes/digitac_bod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; visual mesh filename=../digitac/standard_digitac/digitac_asmb/meshes/digitac_bod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
- added link digitac_tip_link, mass 0.000211579321175967; collision mesh filename=../digitac/standard_digitac/digitac_asmb/meshes/digitac_cor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; visual mesh filename=../digitac/standard_digitac/digitac_asmb_hollow/meshes/digi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
Joints:
- removed joint digit_ee_joint
- removed joint digit_tip_to_body
- added joint tactip_ee_joint: type fixed, parent ee_link, child digitac_body_link, origin xyz=0.0 0.0 0.0 rpy=-3.14 0.0 3.14
- added joint tactip_tip_to_body: type fixed, parent digitac_body_link, child digitac_tip_link, origin xyz=0 0 0 rpy=3.14159265358979 0 -1.5707963267949, axis 0 0 0
- joint tcp_joint: origin xyz=0.0007 0.0 0.040 rpy=0 0 0 -> xyz=0.0007 0.0 0.046 rpy=0 0 0; parent digit_body_link -> digitac_body_link

File: tactile_gym/assets/robot_assets/ur5/ur5_with_standard_digitac.urdf (robot description, URDF)
Before this commit: robot universal_robot, 12 links, 11 joints
Links:
- removed link digit_body_link
- removed link digit_tip_link
- added link digitac_body_link, mass 0.00791827593084163; collision mesh filename=../digitac/standard_digitac/digitac_asmb/meshes/digitac_bod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; visual mesh filename=../digitac/standard_digitac/digitac_asmb/meshes/digitac_bod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
- added link digitac_tip_link, mass 0.000211579321175967; collision mesh filename=../digitac/standard_digitac/digitac_asmb/meshes/digitac_cor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; visual mesh filename=../digitac/standard_digitac/digitac_asmb_hollow/meshes/digi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
Joints:
- removed joint digit_tip_to_body
- added joint tactip_tip_to_body: type fixed, parent digitac_body_link, child digitac_tip_link, origin xyz=0 0 0 rpy=3.14159265358979 0 -1.5707963267949, axis 0 0 0
- joint tactip_ee_joint: child digit_body_link -> digitac_body_link
- joint tcp_joint: origin xyz=0.0007 0.0 0.040 rpy=0 0 0 -> xyz=0.0007 0.0 0.045 rpy=0 0 0; parent digit_body_link -> digitac_body_link
