Commit message: Added DIGIT for pushing task (UR5 and MG400). Successfully trained.

File: tactile_gym/assets/robot_assets/mg400/digit/mg400_with_right_angle_digit.urdf (robot description, URDF)
Before this commit: robot mg400, 13 links, 12 joints
Links:
- removed link digitac_body_link
- removed link digitac_tip_link
- added link digit_body_link, mass 0.0077837104153161; collision mesh filename=../digit/standard_digit/digit_asmb/meshes/digit_body.STL; visual mesh filename=../digit/standard_digit/digit_asmb/meshes/digit_body.STL
- added link digit_tip_link, mass 0.00130411151086353; collision mesh filename=../digit/standard_digit/digit_asmb/meshes/digit_core.STL; visual mesh filename=../digit/standard_digit/digit_asmb_hollow/meshes/digit_core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 scale=1.0 1.0 1.0
Joints:
- removed joint digitac_ee_joint
- removed joint digitac_tip_to_body
- added joint digit_ee_joint: type fixed, parent ee_link, child digit_body_link, origin xyz=0.0 0.0 -0.03 rpy=3.14 -1.57 1.57
- added joint digit_tip_to_body: type fixed, parent digit_body_link, child digit_tip_link, origin xyz=-0.00151521951809463 -1.36251105150219E-05 -0.00415 rpy=-3.14159265358979 0 1.5707963267949, axis 0 0 0
- joint tcp_joint: origin xyz=0.0007 0.0 0.031 rpy=1.57 0 -1.57 -> xyz=0.0007 0.0 0.025 rpy=1.57 0 -1.57; parent digitac_body_link -> digit_body_link
