Commit message: Added TacTip, DIGIT and DigiTac to the MG400 in the vertical surface following task.

File: tactile_gym/assets/robot_assets/mg400/digit/mg400_with_forward_digit.urdf (robot description, URDF)
Before this commit: robot mg400, 13 links, 12 joints
Joints:
- joint digit_ee_joint: origin xyz=0.0 0.0 -0.03 rpy=3.14 -1.57 1.57 -> xyz=0.0 0.0 -0.03 rpy=3.14 -1.57 3.14

File: tactile_gym/assets/robot_assets/mg400/digitac/mg400_with_forward_digitac.urdf (robot description, URDF)
Before this commit: robot mg400, 13 links, 12 joints
Links:
- removed link digit_body_link
- removed link digit_tip_link
- added link digitac_body_link, mass 0.00791827593084163; collision mesh filename=../digitac/standard_digitac/digitac_asmb/meshes/digitac_bod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; visual mesh filename=../digitac/standard_digitac/digitac_asmb/meshes/digitac_bod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
- added link digitac_tip_link, mass 0.000211579321175967; collision mesh filename=../digitac/standard_digitac/digitac_asmb/meshes/digitac_cor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; visual mesh filename=../digitac/standard_digitac/digitac_asmb_hollow/meshes/digi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
Joints:
- removed joint digit_ee_joint
- removed joint digit_tip_to_body
- added joint digitac_ee_joint: type fixed, parent ee_link, child digitac_body_link, origin xyz=0.0 0.0 -0.03 rpy=3.14 -1.57 0
- added joint digitac_tip_to_body: type fixed, parent digitac_body_link, child digitac_tip_link, origin xyz=0 0 0 rpy=3.14159265358979 0 -1.5707963267949, axis 0 0 0
- joint tcp_joint: origin xyz=0.0007 0.0 0.025 rpy=1.57 0 -1.57 -> xyz=0.0007 0.0 0.031 rpy=1.57 0 -1.57; parent digit_body_link -> digitac_body_link

File: tactile_gym/assets/robot_assets/mg400/tactip/mg400_with_forward_tactip.urdf (robot description, URDF)
Before this commit: robot mg400, 13 links, 12 joints
Links:
- removed link digit_body_link
- removed link digit_tip_link
- added link tactip_adapter_link, mass 0.1; collision mesh filename=../tactip/right_angle_tactip/adapter/right_angle_adapter.obj scale=0.7 0.7 0.7; visual mesh filename=../tactip/right_angle_tactip/adapter/right_angle_adapter.obj scale=0.7 0.7 0.7
- added link tactip_body_link, mass 0.25; collision mesh filename=../tactip/standard_tactip/body/tactip_body.obj scale=1.0 1.0 1.0; visual mesh filename=../tactip/standard_tactip/body/tactip_body.obj scale=1.0 1.0 1.0
- added link tactip_tip_link, mass .1; collision mesh filename=../tactip/standard_tactip/tip/core.obj scale=1 1 1; visual mesh filename=../tactip/standard_tactip/tip/skin.obj scale=1.0 1.0 1.0
Joints:
- removed joint digit_ee_joint
- removed joint digit_tip_to_body
- added joint tactip_body_to_adapter: type fixed, parent tactip_adapter_link, child tactip_body_link, origin xyz=0 0 0 rpy=0 0 0
- added joint tactip_ee_joint: type fixed, parent ee_link, child tactip_adapter_link, origin xyz=-0.005 0.00 -0.052 rpy=0 -1.57 -3.14
- added joint tactip_tip_to_body: type fixed, parent tactip_body_link, child tactip_tip_link, origin xyz=0 0 0.065 rpy=1.57 0 0, axis 0 1 0
- joint tcp_joint: origin xyz=0.0007 0.0 0.025 rpy=1.57 0 -1.57 -> xyz=0.0 0.0 0.085 rpy=0 0 0; parent digit_body_link -> tactip_body_link

Commit message: Fixed a bug or the retrain function. Fixed the surface following and pushing tasks. All sensors with MG400 can be trained in the surface task.

File: tactile_gym/assets/robot_assets/mg400/digit/mg400_with_forward_digit.urdf (robot description, URDF)
Before this commit: robot mg400, 13 links, 12 joints
Joints:
- joint digit_ee_joint: origin xyz=0.0 0.0 -0.03 rpy=3.14 -1.57 3.14 -> xyz=0.0 0.0 -0.03 rpy=3.14 -1.57 0
