Commit message: Added MG400 with TacTip and UR5 with DIGIT in the pushing task.

File: tactile_gym/assets/robot_assets/mg400/tactip/mg400_with_right_angle_tactip.urdf (robot description, URDF)
Before this commit: robot mg400, 13 links, 12 joints
Links:
- added link tactip_adapter_link, mass 0.1; collision mesh filename=../tactip/right_angle_tactip/adapter/right_angle_adapter.obj scale=0.7 0.7 0.7; visual mesh filename=../tactip/right_angle_tactip/adapter/right_angle_adapter.obj scale=0.7 0.7 0.7
- link tactip_tip_link: mass 0.01 -> .1
Joints:
- added joint tactip_body_to_adapter: type fixed, parent tactip_adapter_link, child tactip_body_link, origin xyz=0 0 0 rpy=0 0 0
- joint tactip_ee_joint: child tactip_body_link -> tactip_adapter_link; origin xyz=0.0 0.0 0.0 rpy=-3.14 0.0 1.57 -> xyz=0.0 -0.005 -0.052 rpy=0 -1.57 -1.57
- joint tcp_joint: origin xyz=0.0 0.0 0.085 rpy=0 0 -1.57 -> xyz=0.0 0.0 0.085 rpy=0 0 0
