Commit message: update additional robot arms with rest poses, for example_arm_env

File: tactile_gym/assets/robot_assets/franka_panda/digit/franka_panda_with_standard_digit.urdf (robot description, URDF)
Before this commit: robot panda, 13 links, 12 joints
Links:
- removed link tactip_body_link
- removed link tactip_tip_link
- added link digit_body_link, mass 0.0077837104153161; collision mesh filename=../digit/standard_digit/digit_asmb/meshes/digit_body.STL; visual mesh filename=../digit/standard_digit/digit_asmb/meshes/digit_body.STL
- added link digit_tip_link, mass 0.00130411151086353; collision mesh filename=../digit/standard_digit/digit_asmb/meshes/digit_core.STL; visual mesh filename=../digit/standard_digit/digit_asmb_hollow/meshes/digit_core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 scale=1.0 1.0 1.0
- link fixed_base: geometry collision mesh filename=../collision/link0.obj; visual mesh filename=../collision/link0.obj
- link panda_link1: geometry collision mesh filename=../collision/link1.obj; visual mesh filename=visual/link1.obj
- link panda_link2: geometry collision mesh filename=../collision/link2.obj; visual mesh filename=visual/link2.obj
- link panda_link3: geometry collision mesh filename=../collision/link3.obj; visual mesh filename=visual/link3.obj
- link panda_link4: geometry collision mesh filename=../collision/link4.obj; visual mesh filename=visual/link4.obj
- link panda_link5: geometry collision mesh filename=../collision/link5.obj; visual mesh filename=visual/link5.obj
- link panda_link6: geometry collision mesh filename=../collision/link6.obj; visual mesh filename=visual/link6.obj
- link panda_link7: geometry collision mesh filename=../collision/link7.obj; visual mesh filename=../collision/link7.obj
Joints:
- removed joint tactip_ee_joint
- removed joint tactip_tip_to_body
- added joint digit_ee_joint: type fixed, parent ee_link, child digit_body_link, origin xyz=0.0 0.0 0.0 rpy=0.0 0.0 -1.57
- added joint digit_tip_to_body: type fixed, parent digit_body_link, child digit_tip_link, origin xyz=-0.00151521951809463 -1.36251105150219E-05 -0.00415 rpy=-3.14159265358979 0 1.5707963267949, axis 0 0 0
- joint tcp_joint: origin xyz=0.0 0.0 0.085 rpy=0 0 0 -> xyz=0.0007 0.0 0.040 rpy=0 0 0; parent tactip_body_link -> digit_body_link

File: tactile_gym/assets/robot_assets/franka_panda/digitac/franka_panda_with_standard_digitac.urdf (robot description, URDF)
Before this commit: robot panda, 14 links, 13 joints
Links:
- removed link tactip_adapter_link
- removed link tactip_body_link
- removed link tactip_tip_link
- added link digitac_body_link, mass 0.00791827593084163; collision mesh filename=../digitac/standard_digitac/digitac_asmb/meshes/digitac_bod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; visual mesh filename=../digitac/standard_digitac/digitac_asmb/meshes/digitac_bod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
- added link digitac_tip_link, mass 0.000211579321175967; collision mesh filename=../digitac/standard_digitac/digitac_asmb/meshes/digitac_cor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; visual mesh filename=../digitac/standard_digitac/digitac_asmb_hollow/meshes/digi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
- link fixed_base: geometry collision mesh filename=../collision/link0.obj; visual mesh filename=../collision/link0.obj
- link panda_link1: geometry collision mesh filename=../collision/link1.obj; visual mesh filename=visual/link1.obj
- link panda_link2: geometry collision mesh filename=../collision/link2.obj; visual mesh filename=visual/link2.obj
- link panda_link3: geometry collision mesh filename=../collision/link3.obj; visual mesh filename=visual/link3.obj
- link panda_link4: geometry collision mesh filename=../collision/link4.obj; visual mesh filename=visual/link4.obj
- link panda_link5: geometry collision mesh filename=../collision/link5.obj; visual mesh filename=visual/link5.obj
- link panda_link6: geometry collision mesh filename=../collision/link6.obj; visual mesh filename=visual/link6.obj
- link panda_link7: geometry collision mesh filename=../collision/link7.obj; visual mesh filename=../collision/link7.obj
Joints:
- removed joint tactip_body_to_adapter
- removed joint tactip_ee_joint
- added joint digitac_ee_joint: type fixed, parent ee_link, child digitac_body_link, origin xyz=0.0 0.0 0.0 rpy=0.0 0.0 -1.57
- joint tactip_tip_to_body: axis 0 1 0 -> 0 0 0; child tactip_tip_link -> digitac_tip_link; origin xyz=0 0 0.065 rpy=1.57 0 0 -> xyz=0 0 0 rpy=3.14159265358979 0 -1.5707963267949; parent tactip_body_link -> digitac_body_link
- joint tcp_joint: origin xyz=0.0 0.0 0.085 rpy=0 0 0 -> xyz=0.0007 0.0 0.045 rpy=0 0 0; parent tactip_body_link -> digitac_body_link

File: tactile_gym/assets/robot_assets/franka_panda/tactip/franka_panda_with_standard_tactip.urdf (robot description, URDF)
Before this commit: robot panda, 13 links, 12 joints
Links:
- link fixed_base: geometry collision mesh filename=../collision/link0.obj; visual mesh filename=../collision/link0.obj
- link panda_link1: geometry collision mesh filename=../collision/link1.obj; visual mesh filename=visual/link1.obj
- link panda_link2: geometry collision mesh filename=../collision/link2.obj; visual mesh filename=visual/link2.obj
- link panda_link3: geometry collision mesh filename=../collision/link3.obj; visual mesh filename=visual/link3.obj
- link panda_link4: geometry collision mesh filename=../collision/link4.obj; visual mesh filename=visual/link4.obj
- link panda_link5: geometry collision mesh filename=../collision/link5.obj; visual mesh filename=visual/link5.obj
- link panda_link6: geometry collision mesh filename=../collision/link6.obj; visual mesh filename=visual/link6.obj
- link panda_link7: geometry collision mesh filename=../collision/link7.obj; visual mesh filename=../collision/link7.obj
- link tactip_tip_link: geometry collision mesh filename=../tactip/standard_tactip/tip/core.obj scale=1 1 1; visual mesh filename=../tactip/standard_tactip/tip/skin.obj scale=1.0 1.0 1.0
Joints:
- joint tcp_joint: origin xyz=0.0 0.0 0.07 rpy=0 0 0 -> xyz=0.0 0.0 0.085 rpy=0 0 0

File: tactile_gym/assets/robot_assets/ur5/digit/ur5_with_standard_digit.urdf (robot description, URDF)
Before this commit: robot universal_robot, 12 links, 11 joints
Joints:
- removed joint tactip_ee_joint
- added joint digit_ee_joint: type fixed, parent ee_link, child digit_body_link, origin xyz=0.0 0.0 0.0 rpy=-3.14 0.0 3.14

File: tactile_gym/assets/robot_assets/ur5/digitac/ur5_with_standard_digitac.urdf (robot description, URDF)
Before this commit: robot universal_robot, 12 links, 11 joints
Joints:
- removed joint tactip_ee_joint
- added joint digitac_ee_joint: type fixed, parent ee_link, child digitac_body_link, origin xyz=0.0 0.0 0.0 rpy=-3.14 0.0 3.14
